Commit message: This version of pyrobot was pulled September 18, 2019. It was edited to change the following: - Change URDF to match the physical robot as sold by Trossen Robotics - Add new or modified STLs that represent the updated meshes for locobot_description.urdf - Change SRDF to reflect the changes in the updated URDF - Change the rest pose of the arm based on the new physical design - Change the mapToGrid.py to use 'locobot' instead of 'locobase'.

File: robots/LoCoBot/locobot_description/urdf/locobot_description.urdf (robot description, URDF)
Before this commit: robot locobot, 25 links, 24 joints
Links:
- added link battery_link, mass 1.194; collision mesh filename=package://locobot_description/meshes/battery.stl scale=0.001 0.001 0.001; visual mesh filename=package://locobot_description/meshes/battery.stl scale=0.001 0.001 0.001
- link arm_base_link: mass 0.531491686912019 -> 0.379673; geometry collision mesh filename=package://locobot_description/meshes/mobile_base.stl scale=0.001 0.001 0.001; visual mesh filename=package://locobot_description/meshes/mobile_base.stl scale=0.001 0.001 0.001
- link cam_mount: mass 0.508068698311304 -> 2.091937; geometry collision mesh filename=package://locobot_description/meshes/cam_mount.stl scale=0.001 0.001 0.001; visual mesh filename=package://locobot_description/meshes/cam_mount.stl scale=0.001 0.001 0.001
- link plate_1: mass 0.640128902693298 -> 0.27854; geometry collision mesh filename=package://locobot_description/meshes/plate_bottom.stl scale=0.001 0.001 0.001; visual mesh filename=package://locobot_description/meshes/plate_bottom.stl scale=0.001 0.001 0.001
- link plate_2: mass 0.640128902693298 -> 0.27854; geometry collision mesh filename=package://locobot_description/meshes/plate_top.stl scale=0.001 0.001 0.001; visual mesh filename=package://locobot_description/meshes/plate_top.stl scale=0.001 0.001 0.001
Joints:
- added joint battery_link_joint: type fixed, parent plate_2, child battery_link, origin xyz=-0.09703321 0 0.005375 rpy=0 0 0, axis 0 0 0
- joint arm_base_link_joint: origin xyz=0 0 0.001 rpy=0 0 0 -> xyz=0 0 0.002375 rpy=0 0 0
- joint cam_mount_joint: origin xyz=-0.03751 0 0.1331 rpy=0 0 0 -> xyz=-0.03751 0 0.13775 rpy=0 0 0
- joint head_pan_joint: origin xyz=0.0240154841629213 -0.000373468229198185 0.4065 rpy=0 0 0 -> xyz=0.01755 -0.00008 0.3975 rpy=0 0 0
- joint joint_1: origin xyz=0 0 0.072 rpy=0 0 0 -> xyz=0 0 0.0655 rpy=0 0 0
- joint plate_2_joint: origin xyz=0 0 0.0047625 rpy=0 0 0 -> xyz=0 0 0.00475 rpy=0 0 0
